File: v2/pcb/rfid-uhf-wifi-reader/rfid-uhf-wifi-reader.kicad_pcb (KiCad board)
At the start: 2 copper layers, 50 x 50 mm, 23 parts, among them J1 USB_OTG, J2 Conn_01x05, Q1 BSS138, Q2 BSS138, SW1 SW_Push, SW2 SW_Push, U1 ESP32-WROOM-32, U2 AMS1117-3.3, U3 CH340E

Commit message: update ch340c
Parts:
- removed C4, C5: C, Capacitor_SMD:C_0603_1608Metric
- removed D3: LED, LED_SMD:LED_0603_1608Metric
- removed Q1, Q2: BSS138, Package_TO_SOT_SMD:SOT-23
- removed R6: R_Small, Resistor_SMD:R_0603_1608Metric
- removed U3: CH340E, Package_SO:MSOP-10_3x3mm_P0.5mm
- added C6: C, Capacitor_SMD:C_0603_1608Metric, F.Cu at (122.0, 81.5)
- added C7: C, Capacitor_SMD:C_0603_1608Metric, F.Cu at (131.0, 75.0)
- added Q3: BSS138, Package_TO_SOT_SMD:SOT-23, F.Cu at (134.0, 80.2)
- added Q4: BSS138, Package_TO_SOT_SMD:SOT-23, F.Cu at (134.0, 84.0)
- added U4: CH340C, CH340C:SO016, F.Cu at (128.0, 81.6)
- moved R2 9.14 mm to (134.2, 75.0), turned to -90 degrees
- moved R1 6.78 mm to (132.5, 75.0), turned to -90 degrees
Routing:
- net Net-(Q1-G): track 13.5 -> 0.00 mm, vias 2 -> 0
- net Net-(Q3-S): track 0.00 -> 13.0 mm
- net Net-(Q1-S): track 12.6 -> 0.00 mm
- net +3V3: track 73.6 -> 82.1 mm, vias 2 -> 0
- net Net-(Q3-G): track 0.00 -> 6.19 mm
- net GND: track 10.5 -> 4.51 mm, vias 24 -> 23
- net ESP32_IO0: track 38.0 -> 43.4 mm
- net Net-(U3-TNOW): track 3.83 -> 0.00 mm
- net D+: track 12.1 -> 15.6 mm
- net RX-PROG: track 38.2 -> 40.6 mm
- net Net-(D3-A): track 1.92 -> 0.00 mm
- net +5V: track 46.9 -> 48.2 mm
- net VM-RX: track 25.2 -> 26.1 mm
- net D-: track 14.7 -> 15.5 mm
- net VM-EN: track 35.4 -> 36.1 mm
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